Commit message: -

File: src/notspot_description/urdf/spotmicroai.urdf (robot description, URDF)
Before this commit: robot notspot, 24 links, 23 joints
Links:
- link base_inertia: geometry collision box size=0.14 0.11 0.07; visual mesh filename=package://notspot_description/meshes/stl/spot/mainbody.stl scale=0.001 0.001 0.001
- link front_left_foot_link: geometry collision box size=0.026 0.020 0.13; visual mesh filename=package://notspot_description/meshes/stl/spot/lfoot.stl scale=0.001 0.001 0.001
- link front_left_leg_link: geometry collision box size=0.028 0.036 0.109; visual mesh filename=package://notspot_description/meshes/stl/spot/larm.stl scale=0.001 0.001 0.001
- link front_left_leg_link_cover: geometry visual mesh filename=package://notspot_description/meshes/stl/spot/larm_cover.stl scale=0.001 0.001 0.001
- link front_left_shoulder_link: geometry collision box size=0.044 0.038 0.07; visual mesh filename=package://notspot_description/meshes/stl/spot/lshoulder.stl scale=0.001 0.001 0.001
- link front_left_toe_link: geometry collision sphere radius=0.02; visual mesh filename=package://notspot_description/meshes/stl/spot/foot.stl scale=0.001 0.001 0.001
- link front_link: geometry collision box size=0.058 0.11 0.07; visual mesh filename=package://notspot_description/meshes/stl/spot/frontpart.stl scale=0.001 0.001 0.001
- link front_right_foot_link: geometry collision box size=0.026 0.020 0.13; visual mesh filename=package://notspot_description/meshes/stl/spot/rfoot.stl scale=0.001 0.001 0.001
- link front_right_leg_link: geometry collision box size=0.028 0.036 0.109; visual mesh filename=package://notspot_description/meshes/stl/spot/rarm.stl scale=0.001 0.001 0.001
- link front_right_leg_link_cover: geometry visual mesh filename=package://notspot_description/meshes/stl/spot/rarm_cover.stl scale=0.001 0.001 0.001
- link front_right_shoulder_link: geometry collision box size=0.044 0.038 0.07; visual mesh filename=package://notspot_description/meshes/stl/spot/rshoulder.stl scale=0.001 0.001 0.001
- link front_right_toe_link: geometry collision sphere radius=0.02; visual mesh filename=package://notspot_description/meshes/stl/spot/foot.stl scale=0.001 0.001 0.001
- link rear_left_foot_link: geometry collision box size=0.026 0.020 0.13; visual mesh filename=package://notspot_description/meshes/stl/spot/lfoot.stl scale=0.001 0.001 0.001
- link rear_left_leg_link: geometry collision box size=0.028 0.036 0.109; visual mesh filename=package://notspot_description/meshes/stl/spot/larm.stl scale=0.001 0.001 0.001
- link rear_left_leg_link_cover: geometry visual mesh filename=package://notspot_description/meshes/stl/spot/larm_cover.stl scale=0.001 0.001 0.001
- link rear_left_shoulder_link: geometry collision box size=0.044 0.038 0.07; visual mesh filename=package://notspot_description/meshes/stl/spot/lshoulder.stl scale=0.001 0.001 0.001
- link rear_left_toe_link: geometry collision sphere radius=0.02; visual mesh filename=package://notspot_description/meshes/stl/spot/foot.stl scale=0.001 0.001 0.001
- link rear_link: geometry collision box size=0.04 0.11 0.07; visual mesh filename=package://notspot_description/meshes/stl/spot/backpart.stl scale=0.001 0.001 0.001
- link rear_right_foot_link: geometry collision box size=0.026 0.020 0.13; visual mesh filename=package://notspot_description/meshes/stl/spot/rfoot.stl scale=0.001 0.001 0.001
- link rear_right_leg_link: geometry collision box size=0.028 0.036 0.109; visual mesh filename=package://notspot_description/meshes/stl/spot/rarm.stl scale=0.001 0.001 0.001
- link rear_right_leg_link_cover: geometry visual mesh filename=package://notspot_description/meshes/stl/spot/rarm_cover.stl scale=0.001 0.001 0.001
- link rear_right_shoulder_link: geometry collision box size=0.044 0.038 0.07; visual mesh filename=package://notspot_description/meshes/stl/spot/rshoulder.stl scale=0.001 0.001 0.001
- link rear_right_toe_link: geometry collision sphere radius=0.02; visual mesh filename=package://notspot_description/meshes/stl/spot/foot.stl scale=0.001 0.001 0.001
Joints:
- joint front_left_foot: limit lower=-2.59 upper=0.1 effort=1000.0 velocity=0.5 -> lower=-3 upper=3 effort=1000.0 velocity=3
- joint front_left_leg: limit lower=-2.666 upper=1.548 effort=1000.0 velocity=0.5 -> lower=-3 upper=3 effort=1000.0 velocity=3
- joint front_left_shoulder: limit lower=-0.548 upper=0.548 effort=1000.0 velocity=0.7 -> lower=-3 upper=3 effort=1000.0 velocity=3
- joint front_right_foot: limit lower=-2.59 upper=0.1 effort=1000.0 velocity=0.5 -> lower=-3 upper=3 effort=1000.0 velocity=3
- joint front_right_leg: limit lower=-2.666 upper=1.548 effort=1000.0 velocity=0.5 -> lower=-3 upper=3 effort=1000.0 velocity=3
- joint front_right_shoulder: limit lower=-0.548 upper=0.548 effort=1000.0 velocity=0.7 -> lower=-3 upper=3 effort=1000.0 velocity=3
- joint rear_left_foot: limit lower=-2.59 upper=0.1 effort=1000.0 velocity=0.5 -> lower=-3 upper=3 effort=1000.0 velocity=3
- joint rear_left_leg: limit lower=-2.666 upper=1.548 effort=1000.0 velocity=0.5 -> lower=-3 upper=3 effort=1000.0 velocity=3
- joint rear_left_shoulder: limit lower=-0.548 upper=0.548 effort=1000.0 velocity=0.7 -> lower=-3 upper=3 effort=1000.0 velocity=3
- joint rear_right_foot: limit lower=-2.59 upper=0.1 effort=1000.0 velocity=0.5 -> lower=-3 upper=3 effort=1000.0 velocity=3
- joint rear_right_leg: limit lower=-2.666 upper=1.548 effort=1000.0 velocity=0.5 -> lower=-3 upper=3 effort=1000.0 velocity=3
- joint rear_right_shoulder: limit lower=-0.548 upper=0.548 effort=1000.0 velocity=0.7 -> lower=-3 upper=3 effort=1000.0 velocity=3

File: src/notspot_description/urdf/spotmicroai.urdf.xacro (robot description, xacro)
@@ -35,5 +35,5 @@
             <xacro:if value="${left}">
                <geometry>
-                  <mesh filename="package://notspot_description/meshes/stl/lshoulder.stl" scale="0.001 0.001 0.001" />
+                  <mesh filename="package://notspot_description/meshes/stl/spot/lshoulder.stl" scale="0.001 0.001 0.001" />
                </geometry>
                <origin rpy="0 0 3.1416" xyz="0.135 0.0163 -0.0195" />
@@ -41,5 +41,5 @@
             <xacro:unless value="${left}">
                <geometry>
-                  <mesh filename="package://notspot_description/meshes/stl/rshoulder.stl" scale="0.001 0.001 0.001" />
+                  <mesh filename="package://notspot_description/meshes/stl/spot/rshoulder.stl" scale="0.001 0.001 0.001" />
                </geometry>
                <origin rpy="0 0 3.1416" xyz="0.135 0.0938 -0.0205" />
@@ -84,5 +84,5 @@
             <xacro:if value="${left}">
                <geometry>
-                  <mesh filename="package://notspot_description/meshes/stl/larm_cover.stl" scale="0.001 0.001 0.001" />
+                  <mesh filename="package://notspot_description/meshes/stl/spot/larm_cover.stl" scale="0.001 0.001 0.001" />
                </geometry>
                <origin rpy="0 0 3.1416" xyz="0.134 -0.04 -0.0095" />
@@ -90,5 +90,5 @@
             <xacro:unless value="${left}">
                <geometry>
-                  <mesh filename="package://notspot_description/meshes/stl/rarm_cover.stl" scale="0.001 0.001 0.001" />
+                  <mesh filename="package://notspot_description/meshes/stl/spot/rarm_cover.stl" scale="0.001 0.001 0.001" />
                </geometry>
                <origin rpy="0 0 3.1416" xyz="0.134 0.149 -0.0095" />
@@ -101,5 +101,5 @@
             <xacro:if value="${left}">
                <geometry>
-                  <mesh filename="package://notspot_description/meshes/stl/larm.stl" scale="0.001 0.001 0.001" />
+                  <mesh filename="package://notspot_description/meshes/stl/spot/larm.stl" scale="0.001 0.001 0.001" />
                </geometry>
                <origin rpy="0 0 3.1416" xyz="0.134 -0.04 -0.0095" />
@@ -107,5 +107,5 @@
             <xacro:unless value="${left}">
                <geometry>
-                  <mesh filename="package://notspot_description/meshes/stl/rarm.stl" scale="0.001 0.001 0.001" />
+                  <mesh filename="package://notspot_description/meshes/stl/spot/rarm.stl" scale="0.001 0.001 0.001" />
                </geometry>
                <origin rpy="0 0 3.1416" xyz="0.134 0.149 -0.0095" />
@@ -158,5 +158,5 @@
             <xacro:if value="${left}">
                <geometry>
-                  <mesh filename="package://notspot_description/meshes/stl/lfoot.stl" scale="0.001 0.001 0.001" />
+                  <mesh filename="package://notspot_description/meshes/stl/spot/lfoot.stl" scale="0.001 0.001 0.001" />
                </geometry>
                <origin rpy="0 0 3.1416 " xyz="0.1195 -0.04 0.099" />
@@ -164,5 +164,5 @@
             <xacro:unless value="${left}">
                <geometry>
-                  <mesh filename="package://notspot_description/meshes/stl/rfoot.stl" scale="0.001 0.001 0.001" />
+                  <mesh filename="package://notspot_description/meshes/stl/spot/rfoot.stl" scale="0.001 0.001 0.001" />
                </geometry>
                <origin rpy="0 0 3.1416" xyz="0.1195 0.149 0.099" />
@@ -206,5 +206,5 @@
          <visual>
             <geometry>
-               <mesh filename="package://notspot_description/meshes/stl/foot.stl" scale="0.001 0.001 0.001" />
+               <mesh filename="package://notspot_description/meshes/stl/spot/foot.stl" scale="0.001 0.001 0.001" />
             </geometry>
             <origin rpy="0 0.40010 0" xyz="0 -0.01 0.015" />
@@ -246,5 +246,5 @@
       <visual>
          <geometry>
-            <mesh filename="package://notspot_description/meshes/stl/mainbody.stl" scale="0.001 0.001 0.001" />
+            <mesh filename="package://notspot_description/meshes/stl/spot/mainbody.stl" scale="0.001 0.001 0.001" />
          </geometry>
          <material name="black" />
@@ -269,5 +269,5 @@
       <visual>
          <geometry>
-            <mesh filename="package://notspot_description/meshes/stl/backpart.stl" scale="0.001 0.001 0.001" />
+            <mesh filename="package://notspot_description/meshes/stl/spot/backpart.stl" scale="0.001 0.001 0.001" />
          </geometry>
          <origin rpy="0 0 3.1416" xyz="0.042 0.055 -0.0195" />
@@ -295,5 +295,5 @@
       <visual>
          <geometry>
-            <mesh filename="package://notspot_description/meshes/stl/frontpart.stl" scale="0.001 0.001 0.001" />
+            <mesh filename="package://notspot_description/meshes/stl/spot/frontpart.stl" scale="0.001 0.001 0.001" />
          </geometry>
          <origin rpy="0 0 3.1416" xyz="0.042 0.055 -0.0205" />
