Commit message: -

File: src/notspot_description/urdf/notspot.urdf (robot description, URDF)
Before this commit: robot notspot, 17 links, 16 joints
Links:
- link FL1: geometry visual mesh filename=package://notspot_description/meshes/FL1_obj.obj
- link FL2: geometry collision cylinder length=0.125 radius=0.014; visual mesh filename=package://notspot_description/meshes/L2_obj.obj
- link FL3: geometry collision cylinder length=0.06 radius=0.007; visual mesh filename=package://notspot_description/meshes/L3_obj.obj
- link FR1: geometry visual mesh filename=package://notspot_description/meshes/FR1_obj.obj
- link FR2: geometry collision cylinder length=0.125 radius=0.014; visual mesh filename=package://notspot_description/meshes/R2_obj.obj
- link FR3: geometry collision cylinder length=0.06 radius=0.007; visual mesh filename=package://notspot_description/meshes/R3_obj.obj
- link RL1: geometry visual mesh filename=package://notspot_description/meshes/RL1_obj.obj
- link RL2: geometry collision cylinder length=0.125 radius=0.014; visual mesh filename=package://notspot_description/meshes/L2_obj.obj
- link RL3: geometry collision cylinder length=0.06 radius=0.007; visual mesh filename=package://notspot_description/meshes/L3_obj.obj
- link RR1: geometry visual mesh filename=package://notspot_description/meshes/RR1_obj.obj
- link RR2: geometry collision cylinder length=0.125 radius=0.014; visual mesh filename=package://notspot_description/meshes/R2_obj.obj
- link RR3: geometry collision cylinder length=0.06 radius=0.007; visual mesh filename=package://notspot_description/meshes/R3_obj.obj
- link base_link: geometry collision box size=0.25 0.1285 0.055; visual mesh filename=package://notspot_description/meshes/body_obj.obj

Commit message: -

File: src/notspot_description/urdf/notspot.urdf (robot description, URDF)
Before this commit: robot notspot, 17 links, 16 joints
Links:
- link FL1: geometry visual mesh filename=package://notspot_description/meshes/stl/notspot/FL1_obj.obj
- link FL2: geometry collision cylinder length=0.125 radius=0.014; visual mesh filename=package://notspot_description/meshes/stl/notspot/L2_obj.obj
- link FL3: geometry collision cylinder length=0.06 radius=0.007; visual mesh filename=package://notspot_description/meshes/stl/notspot/L3_obj.obj
- link FR1: geometry visual mesh filename=package://notspot_description/meshes/stl/notspot/FR1_obj.obj
- link FR2: geometry collision cylinder length=0.125 radius=0.014; visual mesh filename=package://notspot_description/meshes/stl/notspot/R2_obj.obj
- link FR3: geometry collision cylinder length=0.06 radius=0.007; visual mesh filename=package://notspot_description/meshes/stl/notspot/R3_obj.obj
- link RL1: geometry visual mesh filename=package://notspot_description/meshes/stl/notspot/RL1_obj.obj
- link RL2: geometry collision cylinder length=0.125 radius=0.014; visual mesh filename=package://notspot_description/meshes/stl/notspot/L2_obj.obj
- link RL3: geometry collision cylinder length=0.06 radius=0.007; visual mesh filename=package://notspot_description/meshes/stl/notspot/L3_obj.obj
- link RR1: geometry visual mesh filename=package://notspot_description/meshes/stl/notspot/RR1_obj.obj
- link RR2: geometry collision cylinder length=0.125 radius=0.014; visual mesh filename=package://notspot_description/meshes/stl/notspot/R2_obj.obj
- link RR3: geometry collision cylinder length=0.06 radius=0.007; visual mesh filename=package://notspot_description/meshes/stl/notspot/R3_obj.obj
- link base_link: geometry collision box size=0.25 0.1285 0.055; visual mesh filename=package://notspot_description/meshes/stl/notspot/body_obj.o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
